File: Hardware/EngineGateway/EngineGateway.kicad_sch (KiCad schematic)
At the start: 41 parts

Commit message: Update schematic
Parts:
- removed D? (x6): SM6T6V8A, Diode_SMD:D_SMB, symbol Diode:SM6T6V8A
- removed J?: Conn_01x03_Male, symbol Connector:Conn_01x03_Male
- removed J?: Conn_01x07_Male, symbol Connector:Conn_01x07_Male
- removed U?: LF351N, symbol Amplifier_Operational:LF351N
- added D? (x6): ESD9B3.3ST5G, Diode_SMD:D_SOD-923, symbol Diode:ESD9B3.3ST5G
- added IC?: LTC1841IS8#TR, SOIC127P599X175-8N, symbol SamacSys_Parts:LTC1841IS8#TR
- added IC?: TEENSY_4.0, TEENSY40, symbol SamacSys_Parts:TEENSY_4.0
- added R? (x2): 500K, Resistor_SMD:R_0603_1608Metric_Pad0.98x0.95mm_HandSolder, symbol Device:R_US
- added R? (x3): 33K, Resistor_SMD:R_0603_1608Metric_Pad0.98x0.95mm_HandSolder, symbol Device:R_US
- added R? (x2): 12K, Resistor_SMD:R_0603_1608Metric_Pad0.98x0.95mm_HandSolder, symbol Device:R_US
- J?: footprint (none) -> Connector_PinHeader_2.54mm:PinHeader_1x04_P2.54mm_Vertical
- J?: footprint (none) -> Connector_PinHeader_2.54mm:PinHeader_1x03_P2.54mm_Vertical
- R? (x3): value R_US -> 33K; footprint (none) -> Resistor_SMD:R_0603_1608Metric_Pad0.98x0.95mm_HandSolder
- R? (x4): value R_US -> 6.04K; footprint (none) -> Resistor_SMD:R_0603_1608Metric_Pad0.98x0.95mm_HandSolder
- R? (x2): value R_US -> 100K; footprint (none) -> Resistor_SMD:R_0603_1608Metric_Pad0.98x0.95mm_HandSolder
- R?: value R_US -> 150; footprint (none) -> Resistor_SMD:R_0603_1608Metric_Pad0.98x0.95mm_HandSolder
- R?: value R_US -> 33K; footprint (none) -> Resistor_SMD:R_0603_1608Metric
- R?: value R_US -> 1.5K; footprint (none) -> Resistor_SMD:R_0603_1608Metric_Pad0.98x0.95mm_HandSolder
- R?: value R_US -> 3.3K; footprint (none) -> Resistor_SMD:R_0603_1608Metric_Pad0.98x0.95mm_HandSolder
Connections:
- net +3.3V: now also IC?.31 (3.3V(250_MA_MAX)), IC?.7 (V+), R?.1, R?.1, R?.1
- net +5V: now also IC?.33 (VIN_(3.6_TO_5.5_VOLTS))
- net GND: now also D?.1 (A1), D?.1 (A1), D?.1 (A1), D?.1 (A1), D?.1 (A1), D?.1 (A1), IC?.1 (GND_1), IC?.17 (GND_2), IC?.2 (V-), IC?.28 (21), IC?.32 (GND_3), IC?.34 (GND_4), IC?.5 (IN_B-), IC?.6 (IN_B+), R?.1, R?.2, R?.2
- net at C?.1, R?.1, R?.2: now also D?.2 (A2), IC?.24 (17)
- net at C?.1, R?.1, R?.2: now also D?.2 (A2), IC?.21 (14)
- net at D?.1 (A1), R?.2: now also IC?.27 (20)
- net at C?.1, R?.1, R?.2: now also D?.2 (A2), IC?.22 (15)
- net at C?.1, R?.1, R?.2: now also D?.2 (A2), IC?.25 (18)
- net at C?.1, J?.2 (Pin_2), R?.2: now also D?.2 (A2), IC?.26 (19)
- net at R?.1: now also R?.2
- net at R?.2: now also J?.8 (Pin_8), R?.2; no longer J?.1 (Pin_1)
- net at C?.1, R?.1, R?.2: now also D?.2 (A2), IC?.23 (16)
- net at R?.1: now also J?.1 (Pin_1), R?.2
- new net: IC?.3 (IN_A+), R?.1, R?.1, R?.2
- new net: IC?.1 (OUT_A), IC?.12 (10), R?.2
- new net: IC?.4 (IN_A-), R?.1, R?.2
Other:
- note added: "Analog 6"
- moved on the sheet: R?
